File: 74HC595 Breakout.kicad_pcb (KiCad board)
At the start: 2 copper layers, 114 x 53 mm, 96 parts, among them J1 Conn_01x08, J10 Conn_01x07, J11 Conn_01x02, J2 Conn_01x08, J3 Conn_01x08, J4 Conn_01x08, J5 Conn_01x08, J6 Conn_01x08, J7 Conn_01x08, J8 Conn_01x08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

Commit message: Ground planes
Routing:
- net GND: vias 12 -> 16
- added copper zone on B.Cu, net GND
- added copper zone on F.Cu, net GND
Other:
- board text added: "74HC595 Breakout"
- board text removed: "74HC595 Breakout V1"
Changed lines of the file:
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@@
     (thickness 1.6)
     (drawings 85)
-    (tracks 863)
+    (tracks 871)
     (zones 0)
     (modules 96)
@@
     (aux_axis_origin 0 0)
     (grid_origin 76.2 59.69)
-    (visible_elements FFFFFF5F)
+    (visible_elements FFFFFF7F)
     (pcbplotparams
       (layerselection 0x010fc_ffffffff)
@@
     (effects (font (size 1 1) (thickness 0.15)) (justify left))
   )
-  (gr_text "74HC595\nBreakout V1" (at 186.69 111.125 90) (layer F.SilkS)
+  (gr_text "74HC595\nBreakout" (at 186.69 111.125 90) (layer F.SilkS)
     (effects (font (size 1.5 1.5) (thickness 0.15)) (justify left))
   )
@@
   (segment (start 91.44 62.23) (end 93.345 62.23) (width 0.5) (layer F.Cu) (net 2))
   (segment (start 93.98 85.09) (end 92.71 86.36) (width 0.5) (layer B.Cu) (net 2))
-  (segment (start 93.98 62.865) (end 93.98 85.09) (width 0.5) (layer B.Cu) (net 2))
+  (segment (start 93.98 62.865) (end 93.98 81.28) (width 0.5) (layer B.Cu) (net 2))
   (segment (start 92.3775 62.23) (end 92.3775 64.77) (width 0.5) (layer F.Cu) (net 2))
   (segment (start 91.44 62.23) (end 92.3775 62.23) (width 0.5) (layer F.Cu) (net 2))
   (via (at 117.475 64.77) (size 0.6) (drill 0.3) (layers F.Cu B.Cu) (net 2))
   (segment (start 117.475 74.770002) (end 117.475 64.77) (width 0.5) (layer B.Cu) (net 2))
-  (segment (start 117.475 84.455) (end 117.475 74.770002) (width 0.5) (layer B.Cu) (net 2))
+  (segment (start 117.475 84.455) (end 117.475 81.915) (width 0.5) (layer B.Cu) (net 2))
   (segment (start 115.57 86.36) (end 117.475 84.455) (width 0.5) (layer B.Cu) (net 2))
   (segment (start 117.475 64.77) (end 115.2375 64.77) (width 0.5) (layer F.Cu) (net 2))
   (via (at 140.335 64.77) (size 0.6) (drill 0.3) (layers F.Cu B.Cu) (net 2))
-  (segment (start 140.335 84.455) (end 140.335 64.77) (width 0.5) (layer B.Cu) (net 2))
+  (segment (start 140.335 84.455) (end 140.335 81.915) (width 0.5) (layer B.Cu) (net 2))
   (segment (start 138.43 86.36) (end 140.335 84.455) (width 0.5) (layer B.Cu) (net 2))
   (segment (start 140.335 64.77) (end 138.0975 64.77) (width 0.5) (layer F.Cu) (net 2))
   (via (at 163.195 64.77) (size 0.6) (drill 0.3) (layers F.Cu B.Cu) (net 2))
-  (segment (start 163.195 84.455) (end 163.195 64.77) (width 0.5) (layer B.Cu) (net 2))
+  (segment (start 163.195 84.455) (end 163.195 83.185) (width 0.5) (layer B.Cu) (net 2))
   (segment (start 161.29 86.36) (end 163.195 84.455) (width 0.5) (layer B.Cu) (net 2))
   (segment (start 163.195 64.77) (end 160.9575 64.77) (width 0.5) (layer F.Cu) (net 2))
+  (segment (start 93.98 81.28) (end 93.98 85.09) (width 0.5) (layer B.Cu) (net 2))
+  (via (at 93.98 81.28) (size 0.6) (drill 0.3) (layers F.Cu B.Cu) (net 2))
+  (segment (start 117.475 81.915) (end 117.475 74.770002) (width 0.5) (layer B.Cu) (net 2))
+  (via (at 117.475 81.915) (size 0.6) (drill 0.3) (layers F.Cu B.Cu) (net 2))
+  (segment (start 140.335 81.915) (end 140.335 64.77) (width 0.5) (layer B.Cu) (net 2))
+  (via (at 140.335 81.915) (size 0.6) (drill 0.3) (layers F.Cu B.Cu) (net 2))
+  (segment (start 163.195 83.185) (end 163.195 64.77) (width 0.5) (layer B.Cu) (net 2))
+  (via (at 163.195 83.185) (size 0.6) (drill 0.3) (layers F.Cu B.Cu) (net 2))
   (segment (start 101.2675 63.5) (end 105.41 63.5) (width 0.2) (layer F.Cu) (net 3))
   (segment (start 101.2675 66.04) (end 105.41 66.04) (width 0.2) (layer F.Cu) (net 4))
@@
   (segment (start 137.16 101.6) (end 137.16 94.615) (width 0.2) (layer B.Cu) (net 143))
   (segment (start 137.16 94.615) (end 134.46 94.615) (width 0.2) (layer F.Cu) (net 143))
+  (zone (net 2) (net_name GND) (layer F.Cu) (hatch edge 0.508)
+    (connect_pads (clearance 0.508))
+    (min_thickness 0.254)
+    (fill yes (arc_segments 32) (thermal_gap 0.508) (thermal_bridge_width 0.508))
+    (polygon
+      (pts
+        (xy 76.2 59.69) (xy 190.2 59.69) (xy 190.2 112.69) (xy 76.2 112.69)
+      )
+    )
+  )
+  (zone (net 2) (net_name GND) (layer B.Cu) (hatch edge 0.508)
+    (connect_pads (clearance 0.508))
+    (min_thickness 0.254)
+    (fill yes (arc_segments 32) (thermal_gap 0.508) (thermal_bridge_width 0.508))
+    (polygon
+      (pts
+        (xy 76.2 59.69) (xy 190.2 59.69) (xy 190.2 112.69) (xy 76.2 112.69)
+      )
+    )
+  )
 )
